File: diode-ladder-filter-synth-module-1st-draft.kicad_pcb (KiCad board)
At the start: 4 copper layers, 85.1 x 53.3 mm, 74 parts, among them J1 power, J6 synth-signal-header-10way, M1 imogen-wren-card, U1 TL074, U2 TL074

Commit message: filter updates layoyut attempt 2
Parts:
- moved R27 10.5 mm to (186.2, 61.7)
- moved R3 9.07 mm to (183.9, 85.9)
- moved G*** 5.61 mm to (152.4, 73.4)
- moved R12 4.31 mm to (148.1, 63.0)
- moved FB2 2.54 mm to (125.0, 68.4), turned to 90 degrees
- moved R19 2.54 mm to (132.6, 68.3)
- moved R20 2.54 mm to (135.9, 68.3)
- moved C9 2.51 mm to (129.3, 68.3)
- moved FB1 1.76 mm to (125.0, 79.6), turned to 90 degrees
- moved R4 1.70 mm to (183.1, 61.7)
- moved R9 1.58 mm to (135.9, 79.7)
- moved R13 1.56 mm to (129.0, 79.7)
- moved R14 1.56 mm to (132.6, 79.7)
- moved R21 1.54 mm to (165.9, 81.0)
- moved C3 1.29 mm to (169.2, 81.0)
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Routing:
- net /CV1_IN: track 0.00 -> 119.3 mm, vias 0 -> 1
- net /CV2_IN: track 0.00 -> 97.1 mm, vias 0 -> 1
- net Net-(U1C--): track 0.00 -> 66.5 mm, vias 0 -> 4
- net Net-(D14-A): track 0.00 -> 53.3 mm, vias 0 -> 2
- net Net-(D8-A): track 0.00 -> 49.9 mm, vias 0 -> 2
- net Net-(D13-K): track 0.00 -> 47.5 mm, vias 0 -> 2
- net /AUDIO_OUT: track 0.00 -> 44.3 mm
- net Net-(U2A--): track 0.00 -> 37.7 mm, vias 0 -> 2
- net Net-(D14-K): track 0.00 -> 33.3 mm, vias 0 -> 2
- net Net-(D7-K): track 0.00 -> 31.5 mm, vias 0 -> 2
- net Net-(PT4-Pad3): track 0.00 -> 29.8 mm, vias 0 -> 1
- net Net-(U1B--): track 0.00 -> 26.2 mm, vias 0 -> 2
- net Net-(D7-A): track 0.00 -> 23.6 mm, vias 0 -> 2
- net Net-(U2D-+): track 0.00 -> 23.0 mm
- net Net-(D10-K): track 0.00 -> 21.1 mm, vias 0 -> 2
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- added copper zone on F.Cu, net GND
